File: lab1/lab1/TaskA2.sch (KiCad schematic (older format))
At the start: 4 parts, among them SW1 SW_Push

Commit message: Signed-off-by: Zacharias Tyllström <zache21@hotmail.se>
Parts:
- gave numbers to parts that had none: 1
Changed lines of the file:
@@
 EESchema Schematic File Version 4
+LIBS:lab1-cache
 EELAYER 26 0
 EELAYER END
@@
 Connection ~ 5750 5000
 $Comp
-L Relay:FINDER-40.52 K?
+L Relay:FINDER-40.52 K1
 U 1 1 5CA6366E
 P 5900 4200
-F 0 "K?" H 6530 4246 50  0000 L CNN
+F 0 "K1" H 6530 4246 50  0000 L CNN
 F 1 "FINDER-40.52" H 6530 4155 50  0000 L CNN
 F 2 "Relay_THT:Relay_DPDT_Finder_40.52" H 7250 4170 50  0001 C CNN
