File: lab1/lab1/TaskA3.sch (KiCad schematic (older format))
At the start: 4 parts, among them SW2 SW_Push

Commit message: Signed-off-by: Zacharias Tyllström <zache21@hotmail.se>
Parts:
- gave numbers to parts that had none: 1
Changed lines of the file:
@@
 EESchema Schematic File Version 4
+LIBS:lab1-cache
 EELAYER 26 0
 EELAYER END
@@
 Connection ~ 5550 5050
 $Comp
-L Relay:FINDER-40.52 K?
+L Relay:FINDER-40.52 K2
 U 1 1 5CA6340E
 P 5750 4250
-F 0 "K?" H 6380 4296 50  0000 L CNN
+F 0 "K2" H 6380 4296 50  0000 L CNN
 F 1 "FINDER-40.52" H 6380 4205 50  0000 L CNN
 F 2 "Relay_THT:Relay_DPDT_Finder_40.52" H 7100 4220 50  0001 C CNN
