File: lab1/lab1/TaskA4.sch (KiCad schematic (older format))
At the start: 5 parts

Commit message: Signed-off-by: Zacharias Tyllström <zache21@hotmail.se>
Parts:
- gave numbers to parts that had none: 3
Changed lines of the file:
@@
 EESchema Schematic File Version 4
+LIBS:lab1-cache
 EELAYER 26 0
 EELAYER END
@@
 $EndComp
 $Comp
-L Relay:FINDER-40.52 K?
+L Relay:FINDER-40.52 K3
 U 1 1 5CA6382A
 P 4950 3900
-F 0 "K?" H 5580 3946 50  0000 L CNN
+F 0 "K3" H 5580 3946 50  0000 L CNN
 F 1 "FINDER-40.52" H 5580 3855 50  0000 L CNN
 F 2 "Relay_THT:Relay_DPDT_Finder_40.52" H 6300 3870 50  0001 C CNN
@@
 $EndComp
 $Comp
-L Switch:SW_Push SW?
+L Switch:SW_Push SW4
 U 1 1 5CA63984
 P 4550 3000
-F 0 "SW?" V 4504 3148 50  0000 L CNN
+F 0 "SW4" V 4504 3148 50  0000 L CNN
 F 1 "SW_Push" V 4595 3148 50  0000 L CNN
 F 2 "" H 4550 3200 50  0001 C CNN
@@
 $EndComp
 $Comp
-L Switch:SW_Push_Open SW?
+L Switch:SW_Push_Open SW3
 U 1 1 5CA639E1
 P 4550 2500
-F 0 "SW?" V 4504 2577 50  0000 L CNN
+F 0 "SW3" V 4504 2577 50  0000 L CNN
 F 1 "SW_Push_Open" V 4595 2577 50  0000 L CNN
 F 2 "" H 4550 2700 50  0001 C CNN
